File: TinyWATCH S3 revision P4/KiCAD 7.0.10/TinyWATCH_S3_P4.kicad_pcb (KiCad board)
At the start: 4 copper layers, 29 x 31.4 mm, 117 parts, among them IC2 ESP32-S3-PICO1-N8R2, IC3 XC6194AA03ER-G, IC4 MIC_I2S_ICS-43434, J2 USB_C, J3 Conn_01x18_Pin, Q1 MMBT2222, Q2 MMBT2222, SW1 SW_Push, SW3 SW_Push, SW5 SW_Push, T1 Tab, T3 P-FET, U1 RV-3028-C7, U2 MMC5633NJL, U3 NCP167BMX330TBG, U4 MAX17048G+T10, U6 W25Q80DVUXIE

Commit message: Updated and added new readme cleaned up footprint naming
Parts:
- AF1, AF2, AF3, C1, C10, C11, C12, C13, C14, C15, C16, C17, C18, C19, C2, C20, C22, C23, C24, C25, C26, C27, C29, C3, C30, C31, C32, C33, C5, C6, C8, C9, L1, R1, R11, R12, R13, R14, R15, R16, R17, R18, R19, R2, R20, R21, R22, R23, R24, R25, R26, R27, R28, R29, R3, R30, R31, R33, R4, R5, R6, R7, R8, R9: footprint TinyS3_P3:_0402_SRN -> TinyWATCH_S3:_0402_SRN
- BAT: footprint Unexpected Maker:JST-PICOBLADE -> TinyWATCH_S3:JST-PICOBLADE
- C21, C28, C7: footprint TinyS3_P3:_0603MP -> TinyWATCH_S3:_0603MP
- CHRG2: footprint TinyS3_P3:SOT23-5-SML2 -> TinyWATCH_S3:SOT23-5-SML2
- D1, D10, D11, D2, D4, D9: footprint Unexpected Maker:TVS X1-DFN1006-2 -> TinyWATCH_S3:TVS X1-DFN1006-2
- D5, D6: footprint Unexpected Maker:SOD-523-MSK4010 -> TinyWATCH_S3:SOD-523-MSK4010
- IC2: footprint UnexpectedMaker:QFN56-ESP32-S3-PROD-THIN -> TinyWATCH_S3:QFN56-ESP32-S3-PROD-THIN
- IC3: footprint Unexpected Maker:XC6194BANNERG -> TinyWATCH_S3:XC6194BANNERG
- IC4: footprint Unexpected Maker:SPH0645LM4H -> TinyWATCH_S3:SPH0645LM4H
- J2: footprint Unexpected Maker:USB-C-16P-LESSPASTE-2-FIxed -> TinyWATCH_S3:USB-C-16P-LESSPASTE-2-FIxed
- SP1: footprint Unexpected Maker:MagneticBuzzer_KLJ-4020 -> TinyWATCH_S3:MagneticBuzzer_KLJ-4020
- T3: footprint TinyS3_P3:SOT723 -> TinyWATCH_S3:SOT723
- U$13: footprint Unexpected Maker:ANT_2450AT18B100E -> TinyWATCH_S3:ANT_2450AT18B100E
- U$88: footprint Unexpected Maker:UM_LOGO_NEW_TINY -> TinyWATCH_S3:UM_LOGO_NEW_TINY
- U$88: footprint UnexpectedMaker:UM_LOGO_NEW_SMALL -> TinyWATCH_S3:UM_LOGO_NEW_SMALL
- U1: footprint Unexpected Maker:IC_RV-3028-C7-32.768KHZ-1PPM-TA-QA -> TinyWATCH_S3:IC_RV-3028-C7-32.768KHZ-1PPM-TA-QA
- U3: footprint UnexpectedMaker:VREG_NCP170AMX300TCG -> TinyWATCH_S3:VREG_NCP170AMX300TCG
- U4: footprint Unexpected Maker:MAX17048G_T10_SON50P200X200X80-9N -> TinyWATCH_S3:MAX17048G_T10_SON50P200X200X80-9N
- U6: footprint Unexpected Maker:Flash_W25Q80DVUXIE -> TinyWATCH_S3:Flash_W25Q80DVUXIE
