File: TinyWATCH S3 revision P4/KiCAD 7.0.10/TinyWATCH_S3_P4.kicad_sch (KiCad schematic)
At the start: 100 parts, among them IC1 XC6194AA03ER-G, IC2 ESP32-S3REV0-SILICON, IC4 MIC_I2S_SPH0645, J2 USB_C, J3 Conn_01x18_Pin, Q1 NPN, Q2 NPN, SW1 SW_Push, SW3 SW_Push, SW5 SW_Push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

Commit message: Updated and added new readme cleaned up footprint naming
Parts:
- C13, C32, R21, R22, R23, R24, R5, R7, R8: footprint TinyS3_P3:_0402_SRN -> TinyWATCH_S3:_0402_SRN
- D1, D10, D11, D2, D4, D9: footprint Unexpected Maker:X1-DFN1006-2 -> TinyWATCH_S3:X1-DFN1006-2
- D6: footprint Unexpected Maker:SOD-523-MSK4010 -> TinyWATCH_S3:SOD-523-MSK4010
- IC4: footprint Unexpected Maker:SPH0645LM4H -> TinyWATCH_S3:SPH0645LM4H
- U$13: symbol UnexpectedMaker:NN02-101 -> TinyWATCH_S3:NN02-101
- U1: footprint UnexpectedMaker:IC_RV-3028-C7-32.768KHZ-1PPM-TA-QA -> TinyWATCH_S3:IC_RV-3028-C7-32.768KHZ-1PPM-TA-QA; symbol UnexpectedMaker:RV-3028-C7-32.768KHZ-1PPM-TA-QA -> TinyWATCH_S3:RV-3028-C7-32.768KHZ-1PPM-TA-QA
- U4: footprint Unexpected Maker:MAX17048G_T10_SON50P200X200X80-9N -> TinyWATCH_S3:MAX17048G_T10_SON50P200X200X80-9N
- U5: footprint Unexpected Maker:Flash_W25Q80DVUXIE -> TinyWATCH_S3:Flash_W25Q80DVUXIE
Changed lines of the file:
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@@
       (effects (font (size 1.27 1.27)) (justify right))
     )
-    (property "Footprint" "Unexpected Maker:X1-DFN1006-2" (at 163.703 59.182 0)
+    (property "Footprint" "TinyWATCH_S3:X1-DFN1006-2" (at 163.703 59.182 0)
       (effects (font (size 1.27 1.27)) hide)
     )
@@
       (effects (font (size 1.27 1.27)) (justify right))
     )
-    (property "Footprint" "Unexpected Maker:X1-DFN1006-2" (at 237.49 236.982 0)
+    (property "Footprint" "TinyWATCH_S3:X1-DFN1006-2" (at 237.49 236.982 0)
       (effects (font (size 1.27 1.27)) hide)
     )
@@
       (effects (font (size 1.27 1.0795)) (justify left bottom) hide)
     )
-    (property "Footprint" "Unexpected Maker:SOD-523-MSK4010" (at 47.498 240.03 0)
+    (property "Footprint" "TinyWATCH_S3:SOD-523-MSK4010" (at 47.498 240.03 0)
       (effects (font (size 1.27 1.27)) hide)
     )
@@
       (effects (font (size 1.27 1.27)))
     )
-    (property "Footprint" "TinyS3_P3:_0402_SRN" (at 393.827 198.374 0)
+    (property "Footprint" "TinyWATCH_S3:_0402_SRN" (at 393.827 198.374 0)
       (effects (font (size 1.27 1.27)) hide)
     )
@@
       (effects (font (size 1.27 1.27)) (justify left))
     )
-    (property "Footprint" "TinyS3_P3:_0402_SRN" (at 338.963 61.849 0)
+    (property "Footprint" "TinyWATCH_S3:_0402_SRN" (at 338.963 61.849 0)
       (effects (font (size 1.27 1.27)) hide)
     )
@@
       (effects (font (size 1.27 1.27)))
     )
-    (property "Footprint" "TinyS3_P3:_0402_SRN" (at 55.499 126.492 0)
+    (property "Footprint" "TinyWATCH_S3:_0402_SRN" (at 55.499 126.492 0)
       (effects (font (size 1.27 1.27)) hide)
     )
@@
     )
   )
-  (symbol (lib_id "UnexpectedMaker:NN02-101") (at 98.044 182.626 0) (unit 1)
+  (symbol (lib_id "TinyWATCH_S3:NN02-101") (at 98.044 182.626 0) (unit 1)
     (in_bom yes) (on_board yes) (dnp no)
     (property "Reference" "U$13" (at 98.044 182.626 0)
@@
       (effects (font (size 1.27 1.27)))
     )
-    (property "Footprint" "TinyS3_P3:_0402_SRN" (at 111.887 103.251 0)
+    (property "Footprint" "TinyWATCH_S3:_0402_SRN" (at 111.887 103.251 0)
       (effects (font (size 1.27 1.27)) hide)
     )
@@
       (effects (font (size 1.27 1.27)))
     )
-    (property "Footprint" "TinyS3_P3:_0402_SRN" (at 384.937 195.58 0)
+    (property "Footprint" "TinyWATCH_S3:_0402_SRN" (at 384.937 195.58 0)
       (effects (font (size 1.27 1.27)) hide)
     )
@@
       (effects (font (size 1.27 1.27)) (justify right))
     )
-    (property "Footprint" "Unexpected Maker:X1-DFN1006-2" (at 152.654 59.309 0)
+    (property "Footprint" "TinyWATCH_S3:X1-DFN1006-2" (at 152.654 59.309 0)
       (effects (font (size 1.27 1.27)) hide)
     )
@@
       (effects (font (size 1.778 1.5113)) (justify left top))
     )
-    (property "Footprint" "Unexpected Maker:Flash_W25Q80DVUXIE" (at 268.732 185.801 0)
+    (property "Footprint" "TinyWATCH_S3:Flash_W25Q80DVUXIE" (at 268.732 185.801 0)
       (effects (font (size 1.27 1.27)) hide)
     )
@@
       (effects (font (size 1.27 1.27)) (justify left))
     )
-    (property "Footprint" "TinyS3_P3:_0402_SRN" (at 343.789 61.849 0)
+    (property "Footprint" "TinyWATCH_S3:_0402_SRN" (at 343.789 61.849 0)
       (effects (font (size 1.27 1.27)) hide)
     )
@@
       (effects (font (size 1.27 1.27)) (justify left))
     )
-    (property "Footprint" "TinyS3_P3:_0402_SRN" (at 318.008 48.514 0)
+    (property "Footprint" "TinyWATCH_S3:_0402_SRN" (at 318.008 48.514 0)
       (effects (font (size 1.27 1.27)) hide)
     )
@@
       (effects (font (size 1.27 1.27)))
     )
-    (property "Footprint" "TinyS3_P3:_0402_SRN" (at 392.303 45.085 0)
+    (property "Footprint" "TinyWATCH_S3:_0402_SRN" (at 392.303 45.085 0)
       (effects (font (size 1.27 1.27)) hide)
     )
@@
       (effects (font (size 1.27 1.27)))
     )
-    (property "Footprint" "Unexpected Maker:MAX17048G_T10_SON50P200X200X80-9N" (at 90.551 120.396 0)
+    (property "Footprint" "TinyWATCH_S3:MAX17048G_T10_SON50P200X200X80-9N" (at 90.551 120.396 0)
       (effects (font (size 1.27 1.27)) (justify bottom) hide)
     )
@@
     )
   )
-  (symbol (lib_id "UnexpectedMaker:RV-3028-C7-32.768KHZ-1PPM-TA-QA") (at 348.996 117.983 0) (unit 1)
+  (symbol (lib_id "TinyWATCH_S3:RV-3028-C7-32.768KHZ-1PPM-TA-QA") (at 348.996 117.983 0) (unit 1)
     (in_bom yes) (on_board yes) (dnp no)
     (property "Reference" "U1" (at 348.869 105.664 0)
@@
       (effects (font (size 1.27 1.27)))
     )
-    (property "Footprint" "UnexpectedMaker:IC_RV-3028-C7-32.768KHZ-1PPM-TA-QA" (at 329.692 136.525 0)
+    (property "Footprint" "TinyWATCH_S3:IC_RV-3028-C7-32.768KHZ-1PPM-TA-QA" (at 329.692 136.525 0)
       (effects (font (size 1.27 1.27)) (justify left bottom) hide)
     )
@@
       (effects (font (size 1.27 1.27)) hide)
     )
-    (property "Footprint" "Unexpected Maker:SPH0645LM4H" (at 50.673 198.882 0)
+    (property "Footprint" "TinyWATCH_S3:SPH0645LM4H" (at 50.673 198.882 0)
       (effects (font (size 1.27 1.27)) hide)
     )
@@
       (effects (font (size 1.27 1.27)) (justify right))
     )
-    (property "Footprint" "Unexpected Maker:X1-DFN1006-2" (at 141.224 59.436 0)
+    (property "Footprint" "TinyWATCH_S3:X1-DFN1006-2" (at 141.224 59.436 0)
       (effects (font (size 1.27 1.27)) hide)
     )
@@
       (effects (font (size 1.27 1.27)))
     )
-    (property "Footprint" "TinyS3_P3:_0402_SRN" (at 392.303 62.865 0)
+    (property "Footprint" "TinyWATCH_S3:_0402_SRN" (at 392.303 62.865 0)
       (effects (font (size 1.27 1.27)) hide)
     )
@@
       (effects (font (size 1.27 1.27)))
     )
-    (property "Footprint" "TinyS3_P3:_0402_SRN" (at 329.311 214.122 0)
+    (property "Footprint" "TinyWATCH_S3:_0402_SRN" (at 329.311 214.122 0)
       (effects (font (size 1.27 1.27)) hide)
     )
@@
       (effects (font (size 1.27 1.27)) (justify right))
     )
-    (property "Footprint" "Unexpected Maker:X1-DFN1006-2" (at 263.144 236.474 0)
+    (property "Footprint" "TinyWATCH_S3:X1-DFN1006-2" (at 263.144 236.474 0)
       (effects (font (size 1.27 1.27)) hide)
     )
@@
       (effects (font (size 1.27 1.27)))
     )
-    (property "Footprint" "TinyS3_P3:_0402_SRN" (at 336.931 208.026 0)
+    (property "Footprint" "TinyWATCH_S3:_0402_SRN" (at 336.931 208.026 0)
       (effects (font (size 1.27 1.27)) hide)
     )
@@
       (effects (font (size 1.27 1.27)) (justify left))
     )
-    (property "Footprint" "Unexpected Maker:X1-DFN1006-2" (at 295.148 237.871 0)
+    (property "Footprint" "TinyWATCH_S3:X1-DFN1006-2" (at 295.148 237.871 0)
       (effects (font (size 1.27 1.27)) hide)
     )
@@
       (effects (font (size 1.27 1.27)))
     )
-    (property "Footprint" "TinyS3_P3:_0402_SRN" (at 347.091 195.326 0)
+    (property "Footprint" "TinyWATCH_S3:_0402_SRN" (at 347.091 195.326 0)
       (effects (font (size 1.27 1.27)) hide)
     )
@@
       (effects (font (size 1.27 1.27)))
     )
-    (property "Footprint" "TinyS3_P3:_0402_SRN" (at 66.548 125.476 0)
+    (property "Footprint" "TinyWATCH_S3:_0402_SRN" (at 66.548 125.476 0)
       (effects (font (size 1.27 1.27)) hide)
     )

Commit message: fixed MICRO/PICO Blade connector footrint description
Parts:
- JST-LIPO1: footprint JSTPH2-NO-STENCIL -> Unexpected Maker:JST-PICOBLADE
Changed lines of the file:
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@@
       (effects (font (size 1.27 1.27)) (justify left bottom))
     )
-    (property "Footprint" "JSTPH2-NO-STENCIL" (at 44.069 115.697 0)
+    (property "Footprint" "Unexpected Maker:JST-PICOBLADE" (at 44.069 115.697 0)
       (effects (font (size 1.27 1.27)) hide)
     )
